File: 8088/8088.sch (KiCad schematic (older format))
At the start: 115 parts, among them CON1 BARREL_JACK, P1 U3PA, P10 CONN_01X15, P11 CONN_01X05, P12 CONN_01X05, P13 CONN_01X08, P14 CONN_01X08, P3 U3PB, P4 RX/TX, P5 U4PC, P6 U4PA, P7 U4PB, P8 GND, P9 CONN_01X06, SW1 STEP_CLK, SW2 RESET, SW3 PWR, U1 8284, U10 2114, U11 ULN2803ADWR, U12 74LS14, U13 ULN2803ADWR, U14 ULN2803ADWR, U15 ULN2803ADWR, U16 7805, U2 8088, U3 8755A, U4 8155, U5 8251A, U6 74LS32, U7 74LS138, U8 8282, U9 2114, Y1 12MHz

Commit message: Changed regulator
Parts:
- removed U16: 7805, TO_SOT_Packages_SMD:TO-252-3_TabPin2, symbol 7805-RESCUE-8088
- added C6: 10uF, Capacitors_SMD:C_0805_HandSoldering, symbol C_Small
- added U16: LM1084IT-5.0/NOPB, TO_SOT_Packages_SMD:TO-263-3_TabPin2, symbol LM1084IT-5.0/NOPB
- C4: value 1uF -> 10uF
Connections:
- net +5V: now also C6.1, U16.2 (OUT)
- net GND: now also C6.2, U16.1 (GND)
- net P_IN: now also U16.3 (IN)
Other:
- moved on the sheet: D35, R37
